File: Eagle Files/Bean_revE.brd (EAGLE design)
At the start: 21.7 x 20.3 mm, 16 parts

Commit message: V0.1 Top Board Finished
Parts:
- added C1: 10uF, SparkFun-Capacitors:EIA3216
- added FRAM: MB85RS64V, radiationbean:SO08
- added J1: (no value), SparkFun-Connectors:JST-2-SMD
- added R1: 10K, SparkFun-Resistors:0603-RES
Connections:
- new net CLK: 5.1, FRAM.SCK
- new net CS: 2.1, FRAM.CS
- new net HOLD: FRAM.HOLD, R1.2
- new net MISO: 4.1, FRAM.SO
- new net MOSI: 3.1, FRAM.SI
- new net N$4: RESET.1
- new net N$5: A0.1
- new net N$6: A1.1
- new net N$7: 0.1
- new net VBAT: BAT.1, J1.2
- new net VCC: C1.A, FRAM.VDD, R1.1, VCC.1
- new net WP: FRAM.WP
- net DATA: now also 1.1
- net GND: now also C1.C, FRAM.GND, GND@2.1, GND@3.1, J1.1
Routing:
- net VCC: track 0.00 -> 31.2 mm, vias 0 -> 1
- net GND: track 0.00 -> 21.8 mm, vias 0 -> 2
- net VBAT: track 0.00 -> 21.8 mm, vias 0 -> 1
- net CLK: track 0.00 -> 16.5 mm, vias 0 -> 1
- net CS: track 0.00 -> 16.0 mm
- net DATA: track 0.00 -> 12.7 mm
- net MISO: track 0.00 -> 7.17 mm
- net MOSI: track 0.00 -> 2.93 mm
- net HOLD: track 0.00 -> 2.14 mm
- added copper zone on layer 16, net GND
Other:
- board size 21.7 x 20.3 mm -> 21.8 x 20.3 mm
- board text added: "Top Board"
- board text added: "v0.1"
