File: Eagle Files/Bean_revE.sch (EAGLE design)
At the start: 16 parts

Commit message: V0.1 Top Board Finished
Parts:
- added C1: 10uF, SparkFun-Capacitors:10UF-16V-10%(TANT)
- added FRAM: MB85RS64V, radiationbean:MB85RS64V
- added J1: (no value), SparkFun-Connectors:JST_2MM_MALE
- added R1: 10K, SparkFun-Resistors:10KOHM-1/10W-1%(0603)0603
Connections:
- new net CLK: 5.P$1, FRAM.SCK
- new net CS: 2.P$1, FRAM.CS
- new net HOLD: FRAM.HOLD, R1.2
- new net MISO: 4.P$1, FRAM.SO
- new net MOSI: 3.P$1, FRAM.SI
- new net N$4: RESET.P$1
- new net N$5: A0.P$1
- new net N$6: A1.P$1
- new net N$7: 0.P$1
- new net VBAT: BAT.P$1, J1.+
- new net VCC: C1.+, FRAM.VDD, R1.1, VCC.P$1
- new net WP: FRAM.WP
- net DATA: now also 1.P$1
- net GND: now also C1.-, FRAM.GND, GND@2.P$1, GND@3.P$1, J1.-
Other:
- note added: "OC1A"
