File: Eagle Files/Bottom Board.brd (EAGLE design)
At the start: 21.8 x 20.3 mm, 20 parts

Commit message: Misc Changes
Other:
- board text removed: "Avoid placing copper in antenna keepout"
- board text removed: "Bean Revision E"
- board text removed: "Bottom Silk: bArt"
- board text removed: "Copper Weight: 1oz"
- board text removed: "Corner mill radius: 0.32""
- board text removed: "Finish: ENIG"
- board text removed: "Finished Thickness: 0.062""
- board text removed: "Layers: 2"
- board text removed: "Material: FR4"
- board text removed: "Min Annular Ring: 0.006""
- board text removed: "Min Drill: 0.008""
- board text removed: "Min Spacing: 0.005""
- board text removed: "Min Trace: 0.007""
- board text removed: "P/N: PTD1013012E"
- board text removed: "Rectangular Dimensions: 1.775" x 0.8" (45.09mm x 20.32mm)"
- board text removed: "Rev E"
- board text removed: "Silkscreen Color: Black"
- board text removed: "Silkscreen: Top and Bottom"
- board text removed: "Soldermask Color: 85% white 10% green 5% blue"
- board text removed: "Soldermask: Top and bottom"
- board text removed: "Top Silk: tPlace tArt"
- board text removed: "ck@"
- board text removed: "punchthrough.com"
- board text removed: "ray@"
